File: Hardware/PCB/BUCKCONV.kicad_pcb (KiCad board)
At the start: 2 copper layers, 43 x 21.2 mm, 15 parts, among them U1 LM2596S-ADJ

Commit message: Add files via upload
Routing:
- net Net-(D1-A): track 0.00 -> 2.02 mm
